Commit message: Finished TP2 content, implemented ik

File: src/IN426/in426_desc/xacro/Robot_1/robot_1.xacro (robot description, xacro)
@@ -68,5 +68,5 @@
 		<parent link="base_link"/>
 		<child link="link_1"/>
-		<origin xyz="0 0 ${base_length}"/>
+		<origin xyz="0 0 ${base_length}" rpy = "0 0 ${-pi/2}"/>
 		<axis xyz="0 0 1"/>
 		<limit effort="10" lower="${-pi/2}" upper="${pi/2}" velocity="1"/>
